File: Hardware/OpenTEC.sch (KiCad schematic (older format))
At the start: 49 parts

Commit message: Add I2C connector
Parts:
- added J?: I2C, symbol Connector:Conn_01x04_Male
- added R? (x2): 2.2K, symbol Device:R_US
Connections:
- net +3V3: now also J?.1 (Pin_1), R?.1, R?.1
- net GND: now also J?.4 (Pin_4)
- net I2C_SCL: now also J?.2 (Pin_2), R?.2
- net I2C_SDA: now also J?.3 (Pin_3), R?.2
Other:
- moved on the sheet: H?, J?, RV?
